File: final_pcb/plantpulse_V1/DisplayDevice/DisplayDevice.kicad_pcb (KiCad board)
At the start: 2 copper layers, 169.1 x 87.3 mm, 10 parts, among them J1 SSD1306, J2 LiPo Battery, M1 X27.168

Commit message: Update PCB
Parts:
- added C1: 100nF, Capacitor_SMD:C_0805_2012Metric, F.Cu at (200.6, 62.0)
- S1: value TS-1187A-B-A-B -> Button; footprint TS1187A:SW_TS-1187A-B-A-B -> Button_Switch_THT:SW_PUSH_6mm
- moved S1 4.88 mm to (191.8, 86.2)
Routing:
- net /3V3: track 79.3 -> 88.4 mm
- net /GND: track 55.5 -> 54.7 mm
- net Net-(U1-GPIO44_D7_RX): track 22.7 -> 23.4 mm
